File: PCB/IV_Swinger_2_module/EAGLE/IV_Swinger_2_module.sch (EAGLE design)
At the start: 24 parts, among them J1 

Commit message: Standard (EMR-based) PCB update to RevB
This is RevB of the standard IVS2 EMR-based module version PCB.  It is based on RevB of the SSR-based module version. The main purpose of this revision is to make the SSR and EMR versions as similar as possible, namely:

  - the connections to the binding posts are both on a screw-terminal block on the left end of the board (like SSR version)

  - pads are provided for the bypass diodes (like SSR version)

  - the current-carrying path from the shunt is now isolated in a stub off the ground plane (like SSR version)

  - R3 is now connected to the shunt with a dedicated trace (like SSR version)

  - Connections to EMR are from a second screw-terminal block that is located on the board where the SSRs are in the SSR version

Note that there is nothing "wrong", per se, with the RevA board. This just cleans a few things up and makes it much easier to compare it with the SSR version.
Parts:
- added D1, D2, D3, D4: WIREPAD4,16O1,6, wirepad:WIREPAD4,16O1,6
- added J2: (no value), SparkFun-Connectors:CONN_03-SCREW-5MM
- FH: device con-lsta:FE05-1 -> my_connectors:CONN_04LONGPADS
- RB: device rcl:R-US_0817/22 -> rcl:R-US_0817/7V
- SHUNT: device rcl:R-US_0617/17 -> rcl:R-US_0617/5V
Connections:
- net N10 renamed N14
- net N9 renamed N13
- removed net N2: R1.1, R2.2, R4.1
- removed net N3: A2.6, R6.1
- removed net N8: A1.5, MCP3202.7
- removed net RELAY_NC: J1.2, RB.2
- new net BLEED+: J2.3, RB.1
- new net N15: D2.P, D3.P
- new net N16: C4.1, R3.1, TLV2462.3
- new net N17: RF.2, RG.2, TLV2462.2
- new net PV+: D1.P, J1.2, R1.2
- net +5V: now also FH.3, R6.1; no longer FH.5, R6.2
- net GND: now also D4.P, J1.1, SHUNT.2; no longer SHUNT.1
- net LOAD_CAP+: now also J2.1, J2.2; no longer J1.1
- net LOAD_CAP-: now also RB.2, SHUNT.1; no longer RB.1, SHUNT.2
- net N1: now also A2.6, R6.2; no longer FH.3, R1.2
- net N11: now also R1.1, R2.2, R4.1; no longer C4.1, R3.1, TLV2462.3
- net N12: now also C5.1, R4.2, TLV2462.5; no longer RF.2, RG.2, TLV2462.2
- net N4: now also A1.8, MCP3202.1, R5.1; no longer C5.1, R4.2, TLV2462.5
- net N5: now also A1.7, MCP3202.5; no longer A1.8, MCP3202.1, R5.1
- net N6: now also A1.6, MCP3202.6; no longer A1.7, MCP3202.5
- net N7: now also A1.5, MCP3202.7; no longer A1.6, MCP3202.6
Other:
- note added: "B"
- note added: "Reverse connection bypass diodes (15SQ045)"
- note added: "Screw terminal blocks"
- note added: "→ From PV+"
- note removed: "A"
- note removed: "Screw terminal block"
- note removed: "→ From PV+ / relay NO"
- moved on the sheet: A1, A2, C1, C2, C3, C4, C5, C6, J1, MCP3202, R1, R2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
